File: PCB_piezo-filter_v3.kicad_sch (KiCad schematic)
At the start: 48 parts, among them J1 Conn_01x02_Pin, J2 Conn_01x03_Pin, J3 Conn_01x01_Pin, J4 Conn_01x01_Pin, J5 Conn_01x01_Pin, J6 Conn_01x01_Pin, U1 TL062, U2 TLC2262CP, U3 TLC2262CP

Commit message: pcb connection
Connections:
- net GND: now also J2.1 (Pin_1); no longer J2.3 (Pin_3)
- net at C1.1, C19.2, R1.2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: now also J2.2 (Pin_2); no longer J2.1 (Pin_1)
- net at C20.2, R2.2, U1.2 (-): now also J2.3 (Pin_3); no longer J2.2 (Pin_2)
- net U2_1IN+: no longer names the net of C3.2, R6.1, U2.3 (+)
Other:
- moved on the sheet: J2
Changed lines of the file:
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@@
 	)
 	(junction
+		(at 38.1 95.25)
+		(diameter 0)
+		(color 0 0 0 0)
+	)
+	(junction
 		(at 44.45 125.73)
 		(diameter 0)
@@
 	)
 	(junction
+		(at 38.1 90.17)
+		(diameter 0)
+		(color 0 0 0 0)
+	)
+	(junction
 		(at 140.97 88.9)
 		(diameter 0)
@@
 	)
 	(junction
-		(at 38.1 90.17)
-		(diameter 0)
-		(color 0 0 0 0)
-	)
-	(junction
 		(at 82.55 83.82)
 		(diameter 0)
@@
 		(color 0 0 0 0)
 	)
-	(junction
-		(at 38.1 95.25)
-		(diameter 0)
-		(color 0 0 0 0)
-	)
 	(wire
 		(pts
@@
 	(wire
 		(pts
-			(xy 34.29 95.25) (xy 38.1 95.25)
-		)
-		(stroke
-			(width 0)
-			(type default)
-		)
-	)
-	(wire
-		(pts
 			(xy 71.12 21.59) (xy 71.12 33.02)
 		)
@@
 	(wire
 		(pts
-			(xy 34.29 96.52) (xy 34.29 97.79)
-		)
-		(stroke
-			(width 0)
-			(type default)
-		)
-	)
-	(wire
-		(pts
 			(xy 71.12 44.45) (xy 74.93 44.45)
 		)
@@
 	(wire
 		(pts
-			(xy 86.36 44.45) (xy 86.36 45.72)
+			(xy 38.1 91.44) (xy 38.1 90.17)
 		)
 		(stroke
@@
 	(wire
 		(pts
-			(xy 48.26 54.61) (xy 38.1 54.61)
+			(xy 86.36 44.45) (xy 86.36 45.72)
 		)
 		(stroke
@@
 	(wire
 		(pts
-			(xy 92.71 68.58) (xy 95.25 68.58)
+			(xy 48.26 54.61) (xy 38.1 54.61)
 		)
 		(stroke
@@
 	(wire
 		(pts
-			(xy 63.5 91.44) (xy 63.5 92.71)
+			(xy 92.71 68.58) (xy 95.25 68.58)
 		)
 		(stroke
@@
 	(wire
 		(pts
-			(xy 34.29 90.17) (xy 38.1 90.17)
+			(xy 63.5 91.44) (xy 63.5 92.71)
 		)
 		(stroke
@@
 	(wire
 		(pts
+			(xy 35.56 88.9) (xy 34.29 88.9)
+		)
+		(stroke
+			(width 0)
+			(type default)
+		)
+	)
+	(wire
+		(pts
 			(xy 133.35 80.01) (xy 133.35 88.9)
 		)
@@
 	(wire
 		(pts
-			(xy 86.36 60.96) (xy 88.9 60.96)
+			(xy 38.1 93.98) (xy 38.1 95.25)
 		)
 		(stroke
@@
 	(wire
 		(pts
-			(xy 38.1 81.28) (xy 43.18 81.28)
+			(xy 86.36 60.96) (xy 88.9 60.96)
 		)
 		(stroke
@@
 	(wire
 		(pts
-			(xy 34.29 95.25) (xy 34.29 93.98)
+			(xy 38.1 81.28) (xy 43.18 81.28)
 		)
 		(stroke
@@
 	(wire
 		(pts
+			(xy 34.29 93.98) (xy 38.1 93.98)
+		)
+		(stroke
+			(width 0)
+			(type default)
+		)
+	)
+	(wire
+		(pts
 			(xy 134.62 114.3) (xy 135.89 114.3)
 		)
@@
 	(wire
 		(pts
-			(xy 125.73 106.68) (xy 125.73 114.3)
+			(xy 35.56 87.63) (xy 35.56 88.9)
 		)
 		(stroke
@@
 	(wire
 		(pts
-			(xy 130.81 22.86) (xy 130.81 34.29)
+			(xy 125.73 106.68) (xy 125.73 114.3)
 		)
 		(stroke
@@
 	(wire
 		(pts
-			(xy 86.36 44.45) (xy 90.17 44.45)
+			(xy 130.81 22.86) (xy 130.81 34.29)
 		)
 		(stroke
@@
 	(wire
 		(pts
+			(xy 34.29 91.44) (xy 38.1 91.44)
+		)
+		(stroke
+			(width 0)
+			(type default)
+		)
+	)
+	(wire
+		(pts
 			(xy 38.1 95.25) (xy 40.64 95.25)
 		)
@@
 	(wire
 		(pts
-			(xy 34.29 90.17) (xy 34.29 91.44)
-		)
-		(stroke
-			(width 0)
-			(type default)
-		)
-	)
-	(wire
-		(pts
 			(xy 151.13 88.9) (xy 151.13 101.6)
 		)
@@
 		)
 	)
-	(global_label "U2_1IN+"
-		(shape input)
-		(at 90.17 44.45 0)
-		(fields_autoplaced yes)
-		(effects
-			(font
-				(size 1.27 1.27)
-			)
-			(justify left)
-		)
-		(property "Intersheetrefs" "${INTERSHEET_REFS}"
-			(at 101.38 44.45 0)
-			(effects
-				(font
-					(size 1.27 1.27)
-				)
-				(justify left)
-				(hide yes)
-			)
-		)
-	)
 	(global_label "VGND"
 		(shape output)
@@
 	(symbol
 		(lib_id "Connector:Conn_01x03_Pin")
-		(at 29.21 93.98 0)
+		(at 29.21 91.44 0)
 		(unit 1)
 		(exclude_from_sim no)
@@
 		(on_board yes)
 		(dnp no)
-		(fields_autoplaced yes)
 		(property "Reference" "J2"
-			(at 29.845 86.36 0)
+			(at 29.845 83.82 0)
 			(effects
 				(font
@@
 		)
 		(property "Value" "Conn_01x03_Pin"
-			(at 29.845 88.9 0)
+			(at 27.432 86.106 0)
 			(effects
 				(font
@@
 		)
 		(property "Footprint" "Connector_PinHeader_2.54mm:PinHeader_1x03_P2.54mm_Vertical"
-			(at 29.21 93.98 0)
+			(at 29.21 91.44 0)
 			(effects
 				(font
@@
 		)
 		(property "Datasheet" "~"
-			(at 29.21 93.98 0)
+			(at 29.21 91.44 0)
 			(effects
 				(font
@@
 		)
 		(property "Description" "Generic connector, single row, 01x03, script generated"
-			(at 29.21 93.98 0)
+			(at 29.21 91.44 0)
 			(effects
 				(font
@@
 	)
 	(symbol
+		(lib_id "Device:R")
+		(at 63.5 96.52 0)
+		(unit 1)
+		(exclude_from_sim no)
+		(in_bom yes)
+		(on_board yes)
+		(dnp no)
+		(fields_autoplaced yes)
+		(property "Reference" "R4"
+			(at 66.04 95.2499 0)
+			(effects
+				(font
+					(size 1.27 1.27)
+				)
+				(justify left)
+			)
+		)
+		(property "Value" "100k"
+			(at 66.04 97.7899 0)
+			(effects
+				(font
+					(size 1.27 1.27)
+				)
+				(justify left)
+			)
+		)
+		(property "Footprint" "Resistor_THT:R_Axial_DIN0207_L6.3mm_D2.5mm_P7.62mm_Horizontal"
+			(at 61.722 96.52 90)
+			(effects
+				(font
+					(size 1.27 1.27)
+				)
+				(hide yes)
+			)
+		)
+		(property "Datasheet" "~"
+			(at 63.5 96.52 0)
+			(effects
+				(font
+					(size 1.27 1.27)
+				)
+				(hide yes)
+			)
+		)
+		(property "Description" "Resistor"
+			(at 63.5 96.52 0)
+			(effects
+				(font
+					(size 1.27 1.27)
+				)
+				(hide yes)
+			)
+		)
+		(pin "1"
+		)
+		(pin "2"
+		)
+		(instances
+			(project "PCB_piezo-filter_v3"
+				(path "/b3b86d91-e7b3-4b98-bddd-d81657c3d3ff"
+					(reference "R4")
+					(unit 1)
+				)
+			)
+		)
+	)
+	(symbol
 		(lib_id "Device:C")
 		(at 165.1 72.39 180)
@@
 	(symbol
 		(lib_id "power:GND")
-		(at 34.29 97.79 0)
+		(at 35.56 87.63 180)
 		(unit 1)
 		(exclude_from_sim no)
@@
 		(fields_autoplaced yes)
 		(property "Reference" "#PWR02"
-			(at 34.29 104.14 0)
+			(at 35.56 81.28 0)
 			(effects
 				(font
@@
 		)
 		(property "Value" "GND"
-			(at 34.29 102.87 0)
+			(at 38.1 86.3599 0)
 			(effects
 				(font
 					(size 1.27 1.27)
 				)
+				(justify right)
 			)
 		)
 		(property "Footprint" ""
-			(at 34.29 97.79 0)
+			(at 35.56 87.63 0)
 			(effects
 				(font
@@
 		)
 		(property "Datasheet" ""
-			(at 34.29 97.79 0)
+			(at 35.56 87.63 0)
 			(effects
 				(font
@@
 		)
 		(property "Description" "Power symbol creates a global label with name \"GND\" , ground"
-			(at 34.29 97.79 0)
+			(at 35.56 87.63 0)
 			(effects
 				(font
@@
 					(unit 1)
 				)
-			)
-		)
-	)
-	(symbol
-		(lib_id "Device:R")
-		(at 63.5 96.52 0)
-		(unit 1)
-		(exclude_from_sim no)
-		(in_bom yes)
-		(on_board yes)
-		(dnp no)
-		(fields_autoplaced yes)
-		(property "Reference" "R4"
-			(at 66.04 95.2499 0)
-			(effects
-				(font
-					(size 1.27 1.27)
-				)
-				(justify left)
-			)
-		)
-		(property "Value" "100k"
-			(at 66.04 97.7899 0)
-			(effects
-				(font
-					(size 1.27 1.27)
-				)
-				(justify left)
-			)
-		)
-		(property "Footprint" "Resistor_THT:R_Axial_DIN0207_L6.3mm_D2.5mm_P7.62mm_Horizontal"
-			(at 61.722 96.52 90)
-			(effects
-				(font
-					(size 1.27 1.27)
-				)
-				(hide yes)
-			)
-		)
-		(property "Datasheet" "~"
-			(at 63.5 96.52 0)
-			(effects
-				(font
-					(size 1.27 1.27)
-				)
-				(hide yes)
-			)
-		)
-		(property "Description" "Resistor"
-			(at 63.5 96.52 0)
-			(effects
-				(font
-					(size 1.27 1.27)
-				)
-				(hide yes)
-			)
-		)
-		(pin "1"
-		)
-		(pin "2"
-		)
-		(instances
-			(project "PCB_piezo-filter_v3"
-				(path "/b3b86d91-e7b3-4b98-bddd-d81657c3d3ff"
-					(reference "R4")
-					(unit 1)
-				)
